File: pcb/new1.kicad_pcb (KiCad board)
At the start: 2 copper layers, 66 x 76 mm, 71 parts, among them J1 Conn_01x04_Pin, J4 Screw_Terminal_01x02, J5 Screw_Terminal_01x02, K2 SANYOU_SRD_Form_C, Q1 Q_NPN, SW1 SW_SPST, SW2 SW_SPST, U1 HLW8032, U101 AMS1117-3.3, U2 ESP32-C3-WROOM-02, U3 PC817, U6 PC817, U7 PC817, U8 PC817, U9 LM78M05_TO220

Commit message: Add files via upload
sửa lỗi
Parts:
- moved R24 0.55 mm to (208.0, 79.5), turned to 90 degrees
Routing:
- net /HVL: track 80.6 -> 96.2 mm
- net GND-1: track 158.2 -> 171.1 mm
- net Net-(J5-Pin_1): track 12.1 -> 19.2 mm
- net GND-2: track 164.2 -> 159.9 mm
- net +5V-2: track 0.00 -> 1.55 mm
